File: schematic/hc-sr501/hc-sr501.sch (KiCad schematic (older format))
At the start: 24 parts

Commit message: Avance esquemático
Parts:
- added A?: IRA-S210ST01, TO254P940H490-3, symbol IRA-S210ST01:IRA-S210ST01
- added C? (x2): CP1, symbol Device:CP1
- added D?: D_ALT, symbol Device:D_ALT
- added J?: Conn_01x03, symbol Connector_Generic:Conn_01x03
- added R? (x4): R, symbol Device:R
- added U?: HT7133-1, symbol HT7133-1:HT7133-1
Connections:
- net GND: now also C?.2, C?.2, R?.2, A?.3 (GND), C?.2, C?.2, J?.1 (Pin_1), U?.1 (GND)
- net +3V3: now reaches U?.11 (VDD)
- net +3V3: now also U?.8 (VRF/~RESET), C?.1, R?.1, U?.3 (Vout)
- net at U?.14 (1IN+): now also R?.1
- net at C?.1, C?.2, R?.1: now also U?.16 (1OUT); no longer U?.15 (1IN-)
- net at C?.1, C?.2, R?.1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: now also U?.15 (1IN-); no longer U?.16 (1OUT)
- net at U?.2 (VO): now also R?.2
- net at C?.1: now also R?.1, A?.2 (SOURCE), R?.2
- new net: D?.1 (K), U?.2 (Vin)
- new net: J?.2 (Pin_2), R?.1
- new net: D?.2 (A), J?.3 (Pin_3)
- new net: A?.1 (DRAIN), R?.2
- new net: C?.1, R?.1, R?.2
Other:
- moved on the sheet: C?, R?, RV?, U?

Commit message: Terminado esquematico y asociaciones de footprints
Parts:
- added JP1: Jumper, Jumper:SolderJumper-3_P1.3mm_Bridged2Bar12_Pad1.0x1.5mm_NumberLabels, symbol Jumper:Jumper_3_Bridged12
- A1: renamed from A?; footprint TO254P940H490-3 -> myLib:TO254P940H490-3; symbol IRA-S210ST01:IRA-S210ST01 -> hc-sr501-rescue:IRA-S210ST01-IRA-S210ST01
- C1, C11, C4, C7, C9: renamed from C?; value C -> 10nF; footprint (none) -> Capacitor_SMD:C_0402_1005Metric
- C10, C5: renamed from C?; value C -> 100nF; footprint (none) -> Capacitor_SMD:C_0402_1005Metric
- C12, C6: renamed from C?; value CP1 -> 22uF; footprint (none) -> Capacitor_THT:CP_Radial_D4.0mm_P2.00mm
- C2, C3: renamed from C?; value CP1 -> 47uF; footprint (none) -> Capacitor_THT:CP_Radial_D4.0mm_P2.00mm
- C8: renamed from C?; value C -> 5nF; footprint (none) -> Capacitor_SMD:C_0402_1005Metric
- D1: renamed from D?; footprint (none) -> Diode_SMD:D_MiniMELF
- J1: renamed from J?; value Conn_01x03 -> Conector 3 pines; footprint (none) -> Connector_PinHeader_2.00mm:PinHeader_1x03_P2.00mm_Vertical
- R1, R14: renamed from R?; value R -> 10K; footprint (none) -> Resistor_SMD:R_0402_1005Metric
- R10, R12, R13, R8: renamed from R?; value R -> 1M; footprint (none) -> Resistor_SMD:R_0402_1005Metric
- R11: renamed from R?; footprint (none) -> Resistor_SMD:R_0402_1005Metric
- R15: renamed from R?; value R -> 1K; footprint (none) -> Resistor_SMD:R_0402_1005Metric
- R2, R4, R5: renamed from R?; value R -> 18K; footprint (none) -> Resistor_SMD:R_0402_1005Metric
- R3: renamed from R?; value R -> 47K; footprint (none) -> Resistor_SMD:R_0402_1005Metric
- R6: renamed from R?; value R -> 470K; footprint (none) -> Resistor_SMD:R_0402_1005Metric
- R7: renamed from R?; value R -> 2K; footprint (none) -> Resistor_SMD:R_0402_1005Metric
- R9: renamed from R?; value R -> 6.8K; footprint (none) -> Resistor_SMD:R_0402_1005Metric
- RV1, RV2: renamed from RV?; value R_POT -> 1M; footprint (none) -> Potentiometer_THT:Potentiometer_Bourns_3266X_Horizontal
- U1: renamed from U?; footprint SOIC127P600X180-16N -> myLib:SOIC127P600X180-16N
- U2: renamed from U?; footprint (none) -> Package_TO_SOT_SMD:SOT-89-3; symbol HT7133-1:HT7133-1 -> hc-sr501-rescue:HT7133-1-HT7133-1
Connections:
- net +3V3: now also JP1.1 (A)
- net GND: now also JP1.3 (B)
- net at U1.1 (A): now also JP1.2 (C)
- net 2OUT: now reaches C4.1, RV1.1, RV1.2, U1.12 (2OUT)
- net 2IN-: now reaches C4.2, R6.2, R9.1, U1.13 (2IN-)
- net 1IN+: now reaches R4.1, U1.14 (1IN+)
- net 1IN-: now reaches C7.2, C8.1, R5.1, R8.2, U1.15 (1IN-)
- net 1OUT: now reaches C6.2, C7.1, R8.1, U1.16 (1OUT)
- net Vin: now reaches D1.2 (A), J1.3 (Pin_3)
- net at A1.1 (DRAIN): now also R2.1; no longer R2.2
- net at C2.1, R1.2: now also R2.2; no longer R2.1
Other:
- note added: "Ajuste de retraso"
- note added: "Ajuste sensitividad"
- note added: "Conexiones del CI"
- note added: "Conexiones entre Op-amps del CI"
- note added: "Regulador de voltaje"
- note added: "Sensor PIR"
- moved on the sheet: A1, C1, C10, C11, C12, C2, C3, C4, C5, C6, C7, C8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
