File: schematic/hc-sr501/hc-sr501.kicad_pcb (KiCad board)
At the start: 2 copper layers, 35 x 25 mm, 35 parts, among them J1 Conector 3 pines, U1 BISS0001, U2 HT7133-1

Commit message: Terminado PCB
Parts:
- A1: moved to B.Cu
- moved R15 12.1 mm to (72.5, 44.0), turned to 180 degrees
- moved R4 6.89 mm to (73.0, 48.5)
- moved R2 3.76 mm to (82.5, 47.5)
- moved R6 3.19 mm to (87.7, 55.5)
- moved C1 2.62 mm to (78.0, 52.5)
- moved R12 2.34 mm to (72.5, 51.0)
- moved R11 2.28 mm to (74.0, 51.0)
- moved RV1 2.01 mm to (81.6, 57.2)
- moved C6 2.00 mm to (93.0, 62.0), turned to 180 degrees
- moved U1 1.41 mm to (66.5, 54.0)
- moved R10 1.37 mm to (74.0, 53.5), turned to 90 degrees
- moved C2 0.71 mm to (78.8, 46.4)
- moved R8 0.70 mm to (69.0, 44.8)
- moved R5 0.50 mm to (66.5, 43.0)
- moved C7 0.50 mm to (69.0, 43.0)
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Routing:
- net +3V3: track 0.00 -> 52.8 mm, vias 0 -> 2
- net GND: track 0.00 -> 42.3 mm, vias 0 -> 3
- net /1OUT: track 0.00 -> 38.5 mm, vias 0 -> 1
- net /2IN-: track 0.00 -> 25.9 mm, vias 0 -> 2
- net Net-(C11-Pad1): track 0.00 -> 22.9 mm, vias 0 -> 1
- net /2OUT: track 0.00 -> 21.4 mm, vias 0 -> 1
- net Net-(R15-Pad2): track 0.00 -> 17.4 mm, vias 0 -> 2
- net Net-(R14-Pad2): track 0.00 -> 17.0 mm, vias 0 -> 2
- net Net-(JP1-Pad2): track 0.00 -> 15.8 mm, vias 0 -> 2
- net /1IN-: track 0.00 -> 13.5 mm
- net Net-(A1-Pad2): track 0.00 -> 11.7 mm, vias 0 -> 2
- net Net-(R6-Pad1): track 0.00 -> 11.7 mm, vias 0 -> 1
- net Net-(A1-Pad1): track 0.00 -> 8.45 mm
- net Net-(D1-Pad1): track 0.00 -> 7.59 mm
- net Net-(R12-Pad1): track 0.00 -> 7.54 mm
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- added copper zone on B.Cu, net GND
Other:
- net class Default: clearance 0.2 -> 0.25
- rule trace_clearance: 0.2 -> 0.25
