File: pcb/hc-sr501/hc-sr501.kicad_pcb (KiCad board)
At the start: 2 copper layers, 40.5 x 27.5 mm, 40 parts, among them J1 Conector 3 pines, U1 L78L33_SOT89, U2 BISS0001

Commit message: PCB completo sin montaje
Parts:
- added H5: MountingHole, MountingHole:MountingHole_2.1mm, F.Cu at (157.8, 132.2)
- added H6: MountingHole, MountingHole:MountingHole_2.1mm, F.Cu at (168.0, 132.0)
- moved R9 35.6 mm to (206.5, 129.0)
- moved FID1 30.6 mm to (207.8, 112.0)
- moved C12 23.0 mm to (176.2, 122.2), turned to 90 degrees
- moved C6 20.4 mm to (194.1, 118.5), turned to 0 degrees
- moved C5 16.5 mm to (190.3, 118.5)
- moved R8 15.2 mm to (191.8, 115.5)
- moved JP1 14.8 mm to (185.5, 112.2), turned to 180 degrees
- moved C2 14.5 mm to (206.5, 117.8), turned to 90 degrees
- moved R6 12.6 mm to (189.0, 131.5), turned to 0 degrees
- moved C3 9.20 mm to (199.3, 113.2), turned to 0 degrees
- moved R1 7.99 mm to (203.2, 123.8), turned to 90 degrees
- moved C1 7.81 mm to (193.2, 122.0)
- moved U1 7.21 mm to (200.3, 118.9)
- moved R2 7.14 mm to (200.2, 122.9), turned to 0 degrees
- moved C10 6.19 mm to (176.0, 113.2)
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Routing:
- net +3V3: track 67.7 -> 0.00 mm, vias 3 -> 0
- net Net-(C8-Pad1): track 5.22 -> 34.4 mm, vias 0 -> 2
- net /2IN-: track 44.8 -> 26.9 mm, vias 0 -> 2
- net /1IN-: track 25.9 -> 12.9 mm, vias 2 -> 0
- net Net-(C4-Pad1): track 4.33 -> 17.0 mm, vias 0 -> 1
- net Net-(JP1-Pad2): track 4.14 -> 14.5 mm, vias 0 -> 2
- net GND: track 20.3 -> 29.8 mm, vias 9 -> 6
- net Net-(J1-Pad2): track 4.96 -> 14.3 mm, vias 0 -> 1
- net Net-(R15-Pad2): track 12.7 -> 4.88 mm, vias 2 -> 0
- net /1OUT: track 8.55 -> 15.7 mm
- net Net-(R14-Pad2): track 24.4 -> 17.9 mm
- net Net-(R5-Pad1): track 9.69 -> 4.29 mm
- net Net-(A1-Pad2): track 15.1 -> 9.79 mm
- net Net-(C5-Pad2): track 6.67 -> 1.74 mm
- net Net-(D1-Pad1): track 7.51 -> 2.69 mm
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- added copper zone on F.Cu, net +3V3
Other:
- board size 40.5 x 27.5 mm -> 35 x 25 mm
- board text added: "Ancho de pistas: 0,35 mm"
- board text added: "HC-SR501 v1.0"
- board text added: "IND. ARG"
- board text added: "Margen: 0,3 mm Grilla: 0,25 mm"
- board text added: "Vias: 0,50 mm Pad: 1,00 mm"
- board text removed: "Ancho de pistas: 0.25 mm"
- board text removed: "Ind. Argentina"
- board text removed: "Margen: 0,3 mm Grilla: 0,5 mm"
- board text removed: "Réplica HC-SR501 Ind. Argentina"
- board text removed: "Vias: 0,40 mm Pad: 0,80 mm"

Commit message: Last commit
Parts:
- RV1, RV2: footprint Potentiometer_THT:Potentiometer_Bourns_3266X_Horizontal -> myLib:Potentiometer_Bourns_3362Z_Horizontal
- moved H6 39.8 mm to (206.8, 123.0)
- moved R9 29.0 mm to (177.5, 129.5), turned to 180 degrees
- moved R10 26.3 mm to (180.6, 128.2)
- moved C7 26.1 mm to (177.5, 127.2)
- moved C10 22.2 mm to (184.5, 133.8), turned to 90 degrees
- moved C12 21.2 mm to (196.8, 127.2), turned to 180 degrees
- moved H5 21.1 mm to (176.8, 123.0)
- moved C11 20.2 mm to (194.8, 118.4)
- moved R13 19.3 mm to (191.6, 118.4), turned to 90 degrees
- moved R6 18.5 mm to (175.8, 118.6), turned to 270 degrees
- moved C5 18.1 mm to (205.5, 128.2), turned to 270 degrees
- moved R5 18.0 mm to (176.8, 115.6), turned to 180 degrees
- moved R8 17.2 mm to (203.2, 128.2), turned to 270 degrees
- moved C6 16.8 mm to (207.8, 128.2), turned to 90 degrees
- moved C8 16.3 mm to (177.5, 133.8), turned to 0 degrees
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Routing:
- net Net-(C8-Pad1): track 34.4 -> 4.28 mm, vias 2 -> 0
- net +3V3: track 0.00 -> 25.3 mm, vias 0 -> 1
- net /1IN-: track 12.9 -> 33.4 mm, vias 0 -> 2
- net /2IN-: track 26.9 -> 11.6 mm, vias 2 -> 0
- net Net-(C4-Pad1): track 17.0 -> 4.43 mm, vias 1 -> 0
- net Net-(J1-Pad2): track 14.3 -> 2.87 mm, vias 1 -> 0
- net Net-(A1-Pad1): track 5.19 -> 14.6 mm, vias 0 -> 2
- net Net-(R15-Pad2): track 4.88 -> 13.2 mm, vias 0 -> 2
- net Net-(A1-Pad2): track 9.79 -> 17.7 mm, vias 0 -> 2
- net /1OUT: track 15.7 -> 7.97 mm
- net Net-(R10-Pad1): track 9.59 -> 16.9 mm, vias 0 -> 1
- net GND: track 29.8 -> 36.6 mm, vias 6 -> 5
- net Net-(R14-Pad1): track 3.20 -> 9.22 mm
- net /1IN+: track 2.81 -> 8.63 mm
- net Net-(R14-Pad2): track 17.9 -> 13.6 mm
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Other:
- board text added: "A1"
- board text added: "Margen: 0,5 mm Grilla: 0,25 mm"
- board text removed: "Margen: 0,3 mm Grilla: 0,25 mm"
